File: head.kicad_pcb (KiCad board)
At the start: 2 copper layers, 27.9 x 48.3 mm, 22 parts, among them J1 z probe, J2 HEATER, J3 Conn_01x10, J4 TEMP, J5 COOL_FAN, J6 FAN

Commit message: update,
Parts:
- added G***: LOGO, footprint-lib:logo_icon_4000, F.Cu at (98.4, 75.6)
- moved D4 35.0 mm to (103.3, 71.1), turned to 270 degrees
- moved R4 35.0 mm to (103.3, 71.1), turned to 90 degrees
- moved D3 14.4 mm to (110.9, 71.1), turned to 270 degrees
- moved R3 14.4 mm to (110.9, 71.1), turned to 90 degrees
- moved D2 11.3 mm to (108.3, 71.1), turned to 270 degrees
- moved R2 11.3 mm to (108.3, 71.1), turned to 90 degrees
- moved J4 9.27 mm to (96.8, 67.6), turned to 270 degrees
- moved D1 8.51 mm to (105.8, 71.1), turned to 270 degrees
- moved R1 8.51 mm to (105.8, 71.1), turned to 90 degrees
- moved J2 6.35 mm to (96.8, 58.4)
- moved J6 5.59 mm to (96.8, 49.3)
- moved J5 4.83 mm to (96.8, 40.1)
- moved J1 2.81 mm to (105.4, 37.1)
- moved H3 2.34 mm to (115.2, 75.6)
- moved J3 2.29 mm to (115.6, 41.4)
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Routing:
- net GND: track 146.1 -> 107.2 mm, vias 9 -> 5
- net +5V: track 101.8 -> 69.2 mm, vias 3 -> 0
- net /HOTEND_FAN_P: track 48.3 -> 37.4 mm, vias 3 -> 4
- net /Z_PROBE_SIG: track 28.3 -> 20.2 mm
- net /HOTEND_TEMP_N: track 19.8 -> 26.0 mm
- net /HOTEND_TEMP_P: track 22.3 -> 27.4 mm
- net /PRINT_COOLING_FAN_P: track 50.6 -> 47.6 mm, vias 2 -> 4
- net /HOTEND_HEAT_N: track 44.1 -> 42.1 mm
Other:
- board size 27.9 x 48.3 mm -> 29.7 x 49.8 mm
- board text added: "+"
- board text added: "COOL FAN"
- board text added: "G"
- board text added: "PRO_SIG GND PRO_+ HOT_N TEMP_P TEMP_N GND COOL_P GND FAN_P"
- board text added: "S"
- board text added: "VORON HOTEND PCB"
